File: PCB/harp camera controller.sch (EAGLE design)
At the start: 114 parts, among them IC1 USBLC6-2SC6, IC10 SI8610BC-B-IS, IC2 74LVC1G240DBV, IC3 74LVC1G240DBV, IC4 FT232RL, IC5 TLV70033DDCR, IC6 ATXMEGA32A4U-AU, IC7 SN74LVC1G125DBVT, IC8 SN74LVC1G125DBVT, IC9 TLV70033DDCR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

Commit message: Corrected enable of buffers U2, U3, and U4.
Parts:
- removed R8: 10k, rcl:R-EU_R0402
Connections:
- removed net N$3: R8.2, U2.!3OE
- net +3V3: now also U2.!4OE, U3.!1OE, U3.!2OE, U3.!3OE, U3.!4OE; no longer R8.1
- net GND: now also U2.!3OE; no longer U2.!4OE, U3.!1OE, U3.!2OE, U3.!3OE, U3.!4OE
